File: PCB_CAD_models/adapter.kicad_sch (KiCad schematic)
At the start: 20 parts, among them J1 Conn_01x06, J2 AudioJack3, P1 USB_C_Plug, U1 PCM2902, Y1 12 MHz

Commit message: Update adapter.kicad_sch
Parts:
- C6, C7: value 15pF -> 5.6pF
Changed lines of the file:
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@@
 			)
 		)
-		(property "Value" "15pF"
+		(property "Value" "5.6pF"
 			(at 195.5801 105.41 0)
 			(show_name no)
@@
 			)
 		)
-		(property "Value" "15pF"
+		(property "Value" "5.6pF"
 			(at 195.5801 120.65 0)
 			(show_name no)
